File: kotatsu/kotatsu.kicad_pcb (KiCad board)
At the start: 2 copper layers, 260 x 154.5 mm, 82 parts, among them J1 TRRS_MJ-4PP-9, SW1 SW_Push, SW10 SW_Push, SW11 SW_Push, SW12 SW_Push, SW13 SW_Push, SW14 SW_Push, SW15 SW_Push, SW16 SW_Push, SW17 SW_Push, SW18 SW_Push, SW19 SW_Push, SW2 SW_Push, SW20 SW_Push, SW21 SW_Push, SW22 SW_Push, SW23 SW_Push, SW24 SW_Push, SW25 SW_Push, SW26 SW_Push, SW27 SW_Push, SW28 SW_Push, SW29 SW_Push, SW3 SW_Push, SW30 SW_Push, SW31 SW_Push, SW32 SW_Push, SW33 SW_Push, SW34 SW_Push, SW35 SW_Push, SW36 SW_Push, SW37 SW_Push, SW38 SW_Push, SW39 SW_Push, SW4 SW_Push, SW40 SW_Push, SW5 SW_Push, SW6 SW_Push, SW7 SW_Push, SW8 SW_Push, SW9 SW_Push, U1 Pico

Commit message: right board completed
Routing:
- net row4: track 0.00 -> 337.4 mm
- net col2: track 0.00 -> 293.2 mm
- net row2: track 107.3 -> 393.8 mm
- net GND: track 642.6 -> 915.5 mm
- net row1: track 71.6 -> 300.5 mm
- net col6: track 51.8 -> 279.0 mm
- net col3: track 180.7 -> 348.7 mm
- net row3: track 655.1 -> 809.6 mm
- net col0: track 296.0 -> 440.7 mm
- net row0: track 217.1 -> 356.5 mm
- net col7: track 38.8 -> 148.2 mm
- net col4: track 143.4 -> 244.6 mm
- net col5: track 431.2 -> 515.7 mm
- net col1: track 250.7 -> 333.7 mm
- net Net-(D24-A): track 0.00 -> 54.8 mm
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- added copper zone on B.Cu, net GND
- added copper zone on F.Cu, net GND
